File: hardware/defmon.sch (EAGLE design)
At the start: 18 parts, among them IC2 MEGA8-P, Q1 20MHz, X1 MAB5SH, X2 1503_09

Commit message: Update cad files
Parts:
- removed C1: 100nf, rcl:C-US025-025X050
- removed IC2: MEGA8-P, atmel:MEGA8-P
- removed LED1, LED2: (no value), led:LED3MM
- removed S1: (no value), switch-omron:40-XX
- removed U$1: GB, connector:GB
- removed X1: MAB5SH, con-hirschmann:MAB5SH
- removed X2: 1503_09, con-lumberg:1503_09
- added C6: 100n, rcl:C-USC0603K
- added CONN2: DNP, GenMDMv2:ICSP
- added CONN3: LINK_PORTFINAL, LinkPort by Jazz:LINK_PORTFINAL
- added CU: 10uF, rcl:C-USC0603K
- added DIN: 1X5, header by Jazz:1X5
- added IC1: MEGA8-AI_C16190, atmel:MEGA8-AI
- added JP1: 2X1, header by Jazz:2X1
- added LED3, LED4: C2286, Led by Jazz:0603LED
- added MIDI, TRIG: PJ313, GenMDMv200:PJ313
- added R5, R6: 220Ohms, rcl:R-US_R0603
- added SW1: MODE, Switch by Jazz:TACTILETS5215A
- C2, C3: value 100nf -> 100n; device rcl:C-US025-025X050 -> rcl:C-USC0603K
- C4, C5: device rcl:C-US025-025X050 -> rcl:C-USC0603K
- Q1: value 20MHz -> 20MHz_C172730; device crystal:CRYSTALHC49U-V -> GenMDMv200:CRYSTAL
- R1, R2: value 220 -> 220ohms; device rcl:R-US_0204/7 -> rcl:R-US_R0603
- R3: value 220 -> 220Ohms; device rcl:R-US_0204/7 -> rcl:R-US_R0603
- R4: value 10k -> 10kOhms; device rcl:R-US_0204/7 -> rcl:R-US_R0603
- U$2: value C64U -> CONNECTOR_C64UJ; device connector:C64U -> defmon:CONNECTOR_C64UJ
Connections:
- removed net CLK: IC2.PB0(ICP), U$1.5
- removed net N$13: IC2.PD1(TXD), X1.5
- removed net S_OUT: IC2.PB2(SS/OC1B), U$1.2
- new net !RESET: CONN2.RST, IC1.PC6(/RESET), R4.2
- new net +5V: C3.1, C6.1, CONN2.+V, CU.1, IC1.AVCC, IC1.VCC@1, IC1.VCC@2, R1.2, R3.2, R4.1, U$2.2
- new net GBCLK: CONN3.CLK, IC1.PB0(ICP)
- new net GBSOUT: CONN3.OUT, IC1.PB2(SS/OC1B)
- new net MISO: CONN2.MISO, IC1.PB4(MISO), LED3.A
- new net MOSI: CONN2.MOSI, IC1.PB3(MOSI/OC2), LED4.A
- new net N$20: IC1.PB1(OC1A), SW1.A1, SW1.A2
- new net N$7: LED4.C, R6.1
- new net PC5: DIN.P$1, IC1.PC5(ADC5/SCL)
- new net PD1: DIN.P$5, IC1.PD1(TXD)
- new net SCK: CONN2.SCK, IC1.PB5(SCK)
- net AREF: now also IC1.AREF; no longer IC2.AREF
- net EN: now also IC1.PD6(AIN0); no longer IC2.PD6(AIN0)
- net GND: now also C4.2, C5.2, C6.2, CONN2.GND, CONN3.GND, CU.2, DIN.P$2, IC1.GND, IC1.GND@1, IC1.GND@2, MIDI.2, Q1.GND, R5.2, R6.2, SW1.B1, SW1.B2, TRIG.2; no longer C1.2, C4.1, C5.1, IC2.GND, IC2.GND@1, R1.2, R2.2, S1.P, S1.P1, U$1.6, X1.2, X2.1
- net N$1: now also CONN3.+5V; no longer LED2.C, R2.1
- net N$10: now also IC1.PC4(ADC4/SDA), JP1.1; no longer C1.1, C3.1, IC2.AVCC, IC2.VCC@1, R3.2, R4.1, U$2.2
- net N$11: now also C5.1, IC1.PB7(XTAL2/TOSC2), Q1.X2; no longer C5.2, IC2.PB7(XTAL2/TOSC2), Q1.1
- net N$12: now also MIDI.3, R1.1; no longer IC2.PC6(/RESET), R4.2
- net N$2: now also CONN3.SD; no longer LED1.C, R1.1
- net N$3: now also DIN.P$4; no longer X1.4
- net N$4: now also LED3.C, R5.1; no longer IC2.PB1(OC1A), S1.S
- net N$5: now also CONN3.IN; no longer IC2.PB3(MOSI/OC2), LED2.A
- net N$6: now also MIDI.4, R2.1; no longer IC2.PB4(MISO), LED1.A
- net N$8: now also C4.1, IC1.PB6(XTAL1/TOSC1), Q1.X1; no longer C4.2, IC2.PB6(XTAL1/TOSC1), Q1.2
- net N$9: now also JP1.2, TRIG.3; no longer IC2.PC5(ADC5/SCL), X1.1
- net SYNC: now also IC1.PD5(T1); no longer IC2.PD5(T1)
- net TRIG1: now also IC1.PC0(ADC0), TRIG.4; no longer IC2.PC0(ADC0), X2.2
- net TRIG2: now also DIN.P$3, IC1.PC1(ADC1), R2.2; no longer IC2.PC1(ADC1), X1.3
Other:
- moved on the sheet: C2, C3, C4, C5, R1, R2, R3, R4
